File: Hardware/scope_user_interface.sch (KiCad schematic (older format))
At the start: 110 parts, among them J1 USB_B_Micro, SW1 SW_Push, SW10 SW_Push, SW11 SW_Push, SW12 SW_Push, SW13 SW_Push, SW14 SW_Push, SW18 Rotary_Encoder_Switch, SW19 Rotary_Encoder_Switch, SW2 SW_Push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

Commit message: Changed encoder3b to PB12
Connections:
- net encoder3b: now also U1.1 (b12); no longer U1.30 (a5)
Changed lines of the file:
@@
 Text Label 2600 1800 2    50   ~ 0
 encoder3a
-Text Label 2600 1900 2    50   ~ 0
+Text Label 3800 2600 0    50   ~ 0
 encoder3b
 Text Label 2600 2000 2    50   ~ 0
